Commit message: file update

File: jackal_description/urdf/cam.gazebo.xacro (robot description, xacro)
@@ -1,5 +1,5 @@
 <?xml version="1.0"?>
 <robot name="odean2_sim" xmlns:xacro="http://ros.org/wiki/xacro">
-  <gazebo reference="camera_B_link">
+  <gazebo reference="camera_link">
     <sensor type="camera" name="cam_B">
       <always_on>true</always_on>
@@ -21,5 +21,5 @@
         <updateRate>30.0</updateRate>
         <cameraName>cam_B</cameraName>
-        <frameName>camera_B_link</frameName>
+        <frameName>camera_link</frameName>
         <imageTopicName>rgb/image_raw</imageTopicName>
         <cameraInfoTopicName>rgb/camera_info</cameraInfoTopicName>

File: jackal_description/urdf/cam.urdf.xacro (robot description, xacro)
@@ -2,5 +2,5 @@
 <robot name="odean2" xmlns:xacro="http://ros.org/wiki/xacro">
  <xacro:include filename="$(find test)/urdf/cam.gazebo.xacro"/>
-  <link name="camera_B_link">
+  <link name="camera_link">
     <inertial>
       <origin xyz="0.0076536635969946 -7.04454670178979E-07 -0.000511989237860153" rpy="0 0 0" />
@@ -17,5 +17,5 @@
       <origin xyz="0 0 0" rpy="0 0 0" />
       <geometry>
-        <mesh filename="package://test/meshes/odean2/camera_B_link.STL" />
+        <mesh filename="package://mesh/d435i.STL" />
       </geometry>
       <material name="">
@@ -26,5 +26,5 @@
       <origin xyz="0 0 0" rpy="0 0 0" />
       <geometry>
-        <mesh filename="package://test/meshes/odean2/camera_B_link.STL" />
+        <mesh filename="package://mesh/d435i.STL" />
       </geometry>
     </collision>
